File: SmartFarmMySensors_ArduinoNano.kicad_pcb (KiCad board)
At the start: 2 copper layers, 74 x 52 mm, 14 parts, among them J1 Conn_01x03, J2 Conn_01x03, J3 Conn_01x03, J4 Conn_01x03, J5 Screw_Terminal_01x03, J6 Screw_Terminal_01x03, K1 Relay_SPDT, K2 Relay_SPDT, U1 NRF24L01_Breakout

Commit message: ready to order
Parts:
- added D1: D, Diode_SMD:D_SMA, F.Cu at (146.4, 73.4)
- added D2: D, Diode_SMD:D_SMA, F.Cu at (146.4, 89.4)
- added J7: Power 5V, TerminalBlock:TerminalBlock_Xinya_XY308-2.54-2P_1x02_P2.54mm_Horizontal, F.Cu at (178.6, 64.6)
- added Q1: AO3400A, Package_TO_SOT_SMD:SOT-23, F.Cu at (146.4, 79.7)
- added Q2: AO3400A, Package_TO_SOT_SMD:SOT-23, F.Cu at (146.4, 95.8)
- moved K1 15.0 mm to (153.7, 79.3), turned to 90 degrees
- moved K2 14.7 mm to (153.7, 95.3), turned to 90 degrees
- moved J6 4.13 mm to (178.6, 88.0)
- moved J5 3.45 mm to (178.6, 76.0)
- moved A1 0.27 mm to (137.3, 90.8)
Connections:
- A1 pad 5: RY1 -> RY2
- A1 pad 6: RY2 -> RY1
- K1 pad A2: unconnected-(K1-PadA2) -> +5V
- K2 pad A2: unconnected-(K2-PadA2) -> +5V
Routing:
- net +5V: track 0.00 -> 67.7 mm
- net CO2: track 0.00 -> 28.5 mm
- net CO1: track 0.00 -> 26.9 mm
- net Moisture 4: track 0.00 -> 24.4 mm
- net SCK: track 0.00 -> 21.6 mm
- net RY2: track 0.00 -> 20.8 mm
- net CSN: track 0.00 -> 18.2 mm
- net CE: track 0.00 -> 18.1 mm
- net Moisture 3: track 0.00 -> 18.0 mm
- net NO2: track 0.00 -> 15.8 mm
- net NC1: track 0.00 -> 14.2 mm
- net NO1: track 0.00 -> 14.1 mm
- net NC2: track 0.00 -> 12.9 mm
- net Moisture 2: track 0.00 -> 12.0 mm
- net Moisture 1: track 0.00 -> 11.3 mm
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- added copper zone on F.Cu, net GND
- added copper zone on In1.Cu, net GND
- added copper zone on B.Cu, net VCC
- added copper zone on In2.Cu, net VCC
Other:
- copper layers 2 -> 4
- board text added: "+5V"
- board text added: "A0"
- board text added: "A1"
- board text added: "A2"
- board text added: "A3"
- board text added: "ARDUINO NANO"
- board text added: "COM"
- board text added: "GND"
- board text added: "NC"
- board text added: "NO"
- board text added: "NRF24L01"
- board text added: "POWER"
- board text added: "RELAY1"
- board text added: "RELAY2"
- board text added: "SIET., KMITL."
- board text added: "VCC"
- board text added: "VCC = +3.3V"
